Commit message: Update URDF xacro files for Rizon 10

File: flexiv_description/urdf/rizon.urdf.xacro (robot description, xacro)
@@ -1,11 +1,14 @@
 <?xml version="1.0" encoding="utf-8"?>
-<robot xmlns:xacro="http://www.ros.org/wiki/xacro" name="rizon4">
+<robot xmlns:xacro="http://www.ros.org/wiki/xacro" name="$(arg name)">
   <!-- Enable setting arguments from the launch file -->
+  <xacro:arg name="name" default="rizon"/>
+  <!-- 'rizon_type' values: rizon4, rizon4s, rizon10 -->
   <xacro:arg name="rizon_type" default="rizon4"/>
+  <!-- import main macro -->
+  <xacro:include filename="$(find flexiv_description)/urdf/rizon_macro.xacro"/>
+  <!-- parameters -->
   <xacro:arg name="prefix" default="" />
-  <xacro:include filename="$(find flexiv_description)/urdf/rizon_joints_links.xacro" />
-  <xacro:rizon_joints_links rizon_type="$(arg rizon_type)" prefix="$(arg prefix)" mesh_prefix_path="package://flexiv_description/" />
-  <xacro:include filename="$(find flexiv_description)/urdf/flexiv_arm_materials.xacro" />
-  <xacro:flexiv_arm_materials />
-  <!-- Used for fixing robot -->
+  <xacro:rizon_robot
+    rizon_type="$(arg rizon_type)"
+    prefix="$(arg prefix)"/>
 </robot>

File: flexiv_description/urdf/rizon4_joints_links.xacro (robot description, xacro)
@@ -7,5 +7,5 @@
     NOTE: accurate kinematic but approximated dynamics parameters
   -->
-  <xacro:macro name="rizon_joints_links" params="rizon_type prefix mesh_prefix_path">
+  <xacro:macro name="rizon4_joints_links" params="rizon_type prefix mesh_prefix_path">
     <!-- JOINTS-->
     <joint name="${prefix}base_joint" type="fixed">
@@ -17,5 +17,5 @@
       <parent link="${prefix}base_link"/>
       <child link="${prefix}link1"/>
-      <origin xyz="0.0 0.0 0.155" rpy="0 0 ${pi}"/>
+      <origin xyz="0.0 0.0 0.155" rpy="0 0 ${-pi}"/>
       <axis xyz="0 0 1"/>
       <limit effort="123" lower="-2.7925" upper="2.7925" velocity="2.0944"/>
@@ -80,5 +80,5 @@
         <mass value="3.7" />
         <origin rpy="0 0 0" xyz="0.0 -0.0 0.09" />
-        <inertia ixx="0.019" ixy="0.0" ixz="0.0" iyy="0.02" iyz="0.0" izz="0.009" />
+        <inertia ixx="0.02" ixy="0.0" ixz="0.0" iyy="0.02" iyz="0.0" izz="0.01" />
       </inertial>
       <visual>
@@ -87,9 +87,10 @@
           <mesh filename="${mesh_prefix_path}meshes/${rizon_type}/visual/link0.obj" />
         </geometry>
-      </visual>
-      <collision>
-        <origin xyz="0 0 0" rpy="0 0 0"/>
-        <geometry>
-          <mesh filename="${mesh_prefix_path}meshes/${rizon_type}/collision/link0.obj" />
+        <material name="rizon_light_grey" />
+      </visual>
+      <collision>
+        <origin xyz="0 0 0" rpy="0 0 0"/>
+        <geometry>
+          <mesh filename="${mesh_prefix_path}meshes/${rizon_type}/collision/link0.stl" />
         </geometry>
       </collision>
@@ -99,5 +100,5 @@
         <mass value="3.7" />
         <origin rpy="0 0 0" xyz="0.0 0.01 0.15" />
-        <inertia ixx="0.028" ixy="0.0" ixz="0.0" iyy="0.027" iyz="0.002" izz="0.008" />
+        <inertia ixx="0.03" ixy="0.0" ixz="0.0" iyy="0.03" iyz="0.0" izz="0.01" />
       </inertial>
       <visual>
@@ -106,9 +107,10 @@
           <mesh filename="${mesh_prefix_path}meshes/${rizon_type}/visual/link1.obj" />
         </geometry>
-      </visual>
-      <collision>
-        <origin xyz="0 0 0" rpy="0 0 0" />
-        <geometry>
-          <mesh filename="${mesh_prefix_path}meshes/${rizon_type}/collision/link1.obj" />
+        <material name="rizon_light_grey" />
+      </visual>
+      <collision>
+        <origin xyz="0 0 0" rpy="0 0 0" />
+        <geometry>
+          <mesh filename="${mesh_prefix_path}meshes/${rizon_type}/collision/link1.stl" />
         </geometry>
       </collision>
@@ -118,5 +120,5 @@
         <mass value="2.7" />
         <origin rpy="0 0 0" xyz="0.0 0.04 0.1" />
-        <inertia ixx="0.023" ixy="0.0" ixz="0.0" iyy="0.024" iyz="-0.0" izz="0.004" />
+        <inertia ixx="0.02" ixy="0.0" ixz="0.0" iyy="0.02" iyz="-0.0" izz="0.0" />
       </inertial>
       <visual>
@@ -125,9 +127,10 @@
           <mesh filename="${mesh_prefix_path}meshes/${rizon_type}/visual/link2.obj" />
         </geometry>
-      </visual>
-      <collision>
-        <origin xyz="0 0 0" rpy="0 0 0"/>
-        <geometry>
-          <mesh filename="${mesh_prefix_path}meshes/${rizon_type}/collision/link2.obj" />
+        <material name="rizon_light_grey" />
+      </visual>
+      <collision>
+        <origin xyz="0 0 0" rpy="0 0 0"/>
+        <geometry>
+          <mesh filename="${mesh_prefix_path}meshes/${rizon_type}/collision/link2.stl" />
         </geometry>
       </collision>
@@ -137,5 +140,5 @@
         <mass value="2.4" />
         <origin rpy="0 0 0" xyz="-0.01 -0.0 0.13" />
-        <inertia ixx="0.014" ixy="0.0" ixz="-0.001" iyy="0.014" iyz="-0.001" izz="0.004" />
+        <inertia ixx="0.01" ixy="0.0" ixz="-0.0" iyy="0.01" iyz="-0.0" izz="0.0" />
       </inertial>
       <visual>
@@ -144,9 +147,10 @@
           <mesh filename="${mesh_prefix_path}meshes/${rizon_type}/visual/link3.obj" />
         </geometry>
-      </visual>
-      <collision>
-        <origin xyz="0 0 0" rpy="0 0 0" />
-        <geometry>
-          <mesh filename="${mesh_prefix_path}meshes/${rizon_type}/collision/link3.obj" />
+        <material name="rizon_light_grey" />
+      </visual>
+      <collision>
+        <origin xyz="0 0 0" rpy="0 0 0" />
+        <geometry>
+          <mesh filename="${mesh_prefix_path}meshes/${rizon_type}/collision/link3.stl" />
         </geometry>
       </collision>
@@ -156,5 +160,5 @@
         <mass value="2.4" />
         <origin rpy="0 0 0" xyz="-0.01 0.03 0.1" />
-        <inertia ixx="0.018" ixy="0.0" ixz="-0.002" iyy="0.019" iyz="-0.001" izz="0.003" />
+        <inertia ixx="0.02" ixy="0.0" ixz="-0.0" iyy="0.02" iyz="-0.0" izz="0.0" />
       </inertial>
       <visual>
@@ -163,9 +167,10 @@
           <mesh filename="${mesh_prefix_path}meshes/${rizon_type}/visual/link4.obj" />
         </geometry>
-      </visual>
-      <collision>
-        <origin xyz="0 0 0" rpy="0 0 0"/>
-        <geometry>
-          <mesh filename="${mesh_prefix_path}meshes/${rizon_type}/collision/link4.obj" />
+        <material name="rizon_light_grey" />
+      </visual>
+      <collision>
+        <origin xyz="0 0 0" rpy="0 0 0"/>
+        <geometry>
+          <mesh filename="${mesh_prefix_path}meshes/${rizon_type}/collision/link4.stl" />
         </geometry>
       </collision>
@@ -175,5 +180,5 @@
         <mass value="2.4" />
         <origin rpy="0 0 0" xyz="0.0 0.0 0.13" />
-        <inertia ixx="0.014" ixy="0.0" ixz="0.0" iyy="0.013" iyz="0.001" izz="0.004" />
+        <inertia ixx="0.01" ixy="0.0" ixz="0.0" iyy="0.01" iyz="0.0" izz="0.0" />
       </inertial>
       <visual>
@@ -182,9 +187,10 @@
           <mesh filename="${mesh_prefix_path}meshes/${rizon_type}/visual/link5.obj" />
         </geometry>
-      </visual>
-      <collision>
-        <origin xyz="0 0 0" rpy="0 0 0"/>
-        <geometry>
-          <mesh filename="${mesh_prefix_path}meshes/${rizon_type}/collision/link5.obj" />
+        <material name="rizon_light_grey" />
+      </visual>
+      <collision>
+        <origin xyz="0 0 0" rpy="0 0 0"/>
+        <geometry>
+          <mesh filename="${mesh_prefix_path}meshes/${rizon_type}/collision/link5.stl" />
         </geometry>
       </collision>
@@ -194,5 +200,5 @@
         <mass value="2.1" />
         <origin rpy="0 0 0" xyz="-0.01 0.06 0.07" />
-        <inertia ixx="0.008" ixy="-0.0" ixz="-0.001" iyy="0.009" iyz="0.002" izz="0.004" />
+        <inertia ixx="0.01" ixy="-0.0" ixz="-0.001" iyy="0.01" iyz="0.0" izz="0.0" />
       </inertial>
       <visual>
@@ -201,9 +207,10 @@
           <mesh filename="${mesh_prefix_path}meshes/${rizon_type}/visual/link6.obj" />
         </geometry>
-      </visual>
-      <collision>
-        <origin xyz="0 0 0" rpy="0 0 0"/>
-        <geometry>
-          <mesh filename="${mesh_prefix_path}meshes/${rizon_type}/collision/link6.obj" />
+        <material name="rizon_light_grey" />
+      </visual>
+      <collision>
+        <origin xyz="0 0 0" rpy="0 0 0"/>
+        <geometry>
+          <mesh filename="${mesh_prefix_path}meshes/${rizon_type}/collision/link6.stl" />
         </geometry>
       </collision>
@@ -214,5 +221,5 @@
           <mass value="0.8" />
           <origin rpy="0 0 0" xyz="0.0 0.0 0.03" />
-          <inertia ixx="0.001" ixy="0.0" ixz="0.0" iyy="0.001" iyz="0.0" izz="0.001" />
+          <inertia ixx="0.0" ixy="0.0" ixz="0.0" iyy="0.0" iyz="0.0" izz="0.0" />
         </inertial>
         <visual>
@@ -221,9 +228,10 @@
             <mesh filename="${mesh_prefix_path}meshes/${rizon_type}/visual/link7.obj" />
           </geometry>
+          <material name="rizon_light_grey" />
         </visual>
         <collision>
           <origin xyz="0 0 0" rpy="0 0 0"/>
           <geometry>
-            <mesh filename="${mesh_prefix_path}meshes/${rizon_type}/collision/link7.obj" />
+            <mesh filename="${mesh_prefix_path}meshes/${rizon_type}/collision/link7.stl" />
           </geometry>
         </collision>
@@ -233,5 +241,5 @@
           <mass value="1.4" />
           <origin xyz="0.0 0.0 0.05" rpy="0 0 0"/>
-          <inertia ixx="0.003" iyy="0.003" izz="0.002" ixy="0.0" ixz="0.0" iyz="0.0"/>
+          <inertia ixx="0.0" iyy="0.0" izz="0.0" ixy="0.0" ixz="0.0" iyz="0.0"/>
         </inertial>
         <visual>
@@ -240,9 +248,10 @@
             <mesh filename="${mesh_prefix_path}meshes/${rizon_type}/visual/link7.obj" />
           </geometry>
+          <material name="rizon_light_grey" />
         </visual>
         <collision>
           <origin xyz="0 0 0" rpy="0 0 0"/>
           <geometry>
-            <mesh filename="${mesh_prefix_path}meshes/${rizon_type}/collision/link7.obj" />
+            <mesh filename="${mesh_prefix_path}meshes/${rizon_type}/collision/link7.stl" />
           </geometry>
         </collision>
